File: kicad_files/zx_01.kicad_pcb (KiCad board)
At the start: 2 copper layers, 99.1 x 99.1 mm, 37 parts, among them J1 X1A, J2 X1B, J3 Conn_02x30_Odd_Even

Commit message: .
Other:
- board text added: "*RST/"
- board text removed: "RST/"
Changed lines of the file:
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@@
       (drillshape 0)
       (scaleselection 1)
-      (outputdirectory "gerber")
+      (outputdirectory "../gerber/")
     )
   )
@@
       (effects (font (size 1 1) (thickness 0.15)))
     )
+    (fp_circle (center 0 0) (end 0.5 0) (layer "F.Fab") (width 0.12) (fill none))
     (fp_circle (center 0 0) (end 1 0) (layer "F.Fab") (width 0.12) (fill none))
-    (fp_circle (center 0 0) (end 0.5 0) (layer "F.Fab") (width 0.12) (fill none))
     (pad " " thru_hole circle (at 0 0) (size 5 5) (drill 3) (layers F&B.Cu *.Mask))
     (model "${KICAD6_3DMODEL_DIR}/Connector_Pin.3dshapes/Pin_D1.0mm_L10.0mm.wrl" hide
@@
       (effects (font (size 1 1) (thickness 0.15)))
     )
+    (fp_circle (center 0 0) (end 0.5 0) (layer "F.Fab") (width 0.12) (fill none))
     (fp_circle (center 0 0) (end 1 0) (layer "F.Fab") (width 0.12) (fill none))
-    (fp_circle (center 0 0) (end 0.5 0) (layer "F.Fab") (width 0.12) (fill none))
     (pad " " thru_hole circle (at 0 0) (size 5 5) (drill 3) (layers F&B.Cu *.Mask))
     (model "${KICAD6_3DMODEL_DIR}/Connector_Pin.3dshapes/Pin_D1.0mm_L10.0mm.wrl" hide
@@
     (effects (font (size 1 0.8) (thickness 0.15)) (justify mirror))
   )
-  (gr_text "RST/" (at 102.188423 129.713303 90) (layer "B.SilkS")
+  (gr_text "*RST/" (at 102.188423 129.713303 90) (layer "B.SilkS")
     (effects (font (size 1 0.8) (thickness 0.15)) (justify mirror))
   )
@@
     (effects (font (size 1 0.7) (thickness 0.15)))
   )
-  (gr_text "RST/" (at 102.235 130.175 90) (layer "F.SilkS")
+  (gr_text "*RST/" (at 102.235 130.175 90) (layer "F.SilkS")
     (effects (font (size 1 0.8) (thickness 0.15)))
   )
